File: Nixie_Module_IN-12.sch (KiCad schematic (older format))
At the start: 43 parts, among them J1 CONN_01X07, J3 CONN_01X02, J4 CONN_01X02, Q1 Q_NPN_BEC, Q10 Q_NPN_BEC, Q11 Q_NPN_BEC, Q2 Q_NPN_BEC, Q3 Q_NPN_BEC, Q4 Q_NPN_BEC, Q5 Q_NPN_BEC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

Commit message: Add documentation
Parts:
- C1, C3: value 47u -> 4.7u
- J1: symbol conn:Conn_01x07_Male -> Nixie_Module_IN-12-rescue:Conn_01x07_Male-conn
- J3, J4: symbol conn:Conn_01x02_Male -> Nixie_Module_IN-12-rescue:Conn_01x02_Male-conn
- R1: value 15k -> 47k
Changed lines of the file:
@@
 P 2550 1450
 F 0 "R1" V 2630 1450 50  0000 C CNN
-F 1 "15k" V 2550 1450 50  0000 C CNN
+F 1 "47k" V 2550 1450 50  0000 C CNN
 F 2 "R_SMD:R_0603" V 2480 1450 50  0001 C CNN
 F 3 "" H 2550 1450 50  0001 C CNN
@@
 P 1900 5750
 F 0 "C1" H 1925 5850 50  0000 L CNN
-F 1 "47u" H 1925 5650 50  0000 L CNN
+F 1 "4.7u" H 1925 5650 50  0000 L CNN
 F 2 "C_SMD:C_0603" H 1938 5600 50  0001 C CNN
 F 3 "" H 1900 5750 50  0001 C CNN
@@
 NIX_1
 $Comp
-L conn:Conn_01x02_Male J3
+L Nixie_Module_IN-12-rescue:Conn_01x02_Male-conn J3
 U 1 1 5B6BFF15
 P 10650 5250
@@
 $EndComp
 $Comp
-L conn:Conn_01x02_Male J4
+L Nixie_Module_IN-12-rescue:Conn_01x02_Male-conn J4
 U 1 1 5B6C02A2
 P 10650 5800
@@
 P 1000 4050
 F 0 "C3" H 1025 4150 50  0000 L CNN
-F 1 "47u" H 1025 3950 50  0000 L CNN
+F 1 "4.7u" H 1025 3950 50  0000 L CNN
 F 2 "C_SMD:C_0603" H 1038 3900 50  0001 C CNN
 F 3 "" H 1000 4050 50  0001 C CNN
@@
 NoConn ~ 5050 6900
 $Comp
-L conn:Conn_01x07_Male J1
+L Nixie_Module_IN-12-rescue:Conn_01x07_Male-conn J1
 U 1 1 5B997804
 P 9600 5650

Commit message: add docs
Parts:
- removed U1: SK6812mini, FidgetSpinner:SK6812MINI, symbol FidgetSpinner_SK6812mini_v2-cache:SK6812mini
- added LED1: WS2812B, WS2812b:WS2812B, symbol WS2812b:WS2812B
Connections:
- net +5V: now also LED1.1 (VCC)
- net GND: now also LED1.3 (GND)
- net LED_DIN: now also LED1.4 (DIN)
- net LED_DOUT: now also LED1.2 (DOUT)
Changed lines of the file:
@@
 PCA9685 must be configured as "Direct LED Connection" mode\nINVRT = 1\nOUTDRV = 0
-$Comp
-L FidgetSpinner_SK6812mini_v2-cache:SK6812mini U1
-U 1 1 5B980119
-P 2050 3750
-F 0 "U1" H 2050 3847 60  0000 C CNN
-F 1 "SK6812mini" H 2050 3741 60  0000 C CNN
-F 2 "FidgetSpinner:SK6812MINI" H 2050 3750 60  0001 C CNN
-F 3 "" H 2050 3750 60  0000 C CNN
-	1    2050 3750
-	1    0    0    -1
-$EndComp
 $Comp
 L power:+5V #PWR026
 U 1 1 5B980467
-P 1400 3800
-F 0 "#PWR026" H 1400 3650 50  0001 C CNN
-F 1 "+5V" H 1400 3940 50  0000 C CNN
-F 2 "" H 1400 3800 50  0001 C CNN
-F 3 "" H 1400 3800 50  0001 C CNN
-	1    1400 3800
+P 1600 3700
+F 0 "#PWR026" H 1600 3550 50  0001 C CNN
+F 1 "+5V" H 1600 3840 50  0000 C CNN
+F 2 "" H 1600 3700 50  0001 C CNN
+F 3 "" H 1600 3700 50  0001 C CNN
+	1    1600 3700
 	1    0    0    -1
 $EndComp
@@
 L power:GND #PWR027
 U 1 1 5B9804BE
-P 2700 4200
-F 0 "#PWR027" H 2700 3950 50  0001 C CNN
-F 1 "GND" H 2700 4050 50  0000 C CNN
-F 2 "" H 2700 4200 50  0001 C CNN
-F 3 "" H 2700 4200 50  0001 C CNN
-	1    2700 4200
-	1    0    0    -1
-$EndComp
-Wire Wire Line
-	1500 3900 1400 3900
-Wire Wire Line
-	1400 3900 1400 3800
+P 2800 4450
+F 0 "#PWR027" H 2800 4200 50  0001 C CNN
+F 1 "GND" H 2800 4300 50  0000 C CNN
+F 2 "" H 2800 4450 50  0001 C CNN
+F 3 "" H 2800 4450 50  0001 C CNN
+	1    2800 4450
+	1    0    0    -1
+$EndComp
+Wire Wire Line
+	1700 3800 1600 3800
+Wire Wire Line
+	1600 3800 1600 3700
 $Comp
 L Device:C C3
@@
 	1000 4200 1000 4350
 Wire Wire Line
-	1500 4000 1250 4000
-Wire Wire Line
-	2600 3900 2700 3900
-Wire Wire Line
-	2700 3900 2700 4200
-Wire Wire Line
-	2600 4000 2950 4000
-Text Label 1250 4000 0    50   ~ 0
+	2700 3800 2950 3800
+Wire Wire Line
+	2700 4200 2800 4200
+Wire Wire Line
+	1700 4200 1350 4200
+Text Label 2950 3800 2    50   ~ 0
 LED_DIN
-Text Label 2950 4000 0    50   ~ 0
+Text Label 1350 4200 2    50   ~ 0
 LED_DOUT
 Wire Wire Line
@@
 	-1   0    0    -1
 $EndComp
+$Comp
+L WS2812b:WS2812B LED1
+U 1 1 5C239957
+P 2200 4000
+F 0 "LED1" H 2200 4487 60  0000 C CNN
+F 1 "WS2812B" H 2200 4381 60  0000 C CNN
+F 2 "WS2812b:WS2812B" V 2150 4000 60  0001 C CNN
+F 3 "" V 2150 4000 60  0000 C CNN
+	1    2200 4000
+	1    0    0    -1
+$EndComp
+Wire Wire Line
+	2800 4200 2800 4450
 $EndSCHEMATC
